File: opus/pcb/opus.sch (KiCad schematic (older format))
At the start: 85 parts, among them K000 KEYSW, K001 KEYSW, K002 KEYSW, K003 KEYSW, K004 KEYSW, K005 KEYSW, K006 KEYSW, K007 KEYSW, K008 KEYSW, K009 KEYSW, K010 KEYSW, K011 KEYSW, K100 KEYSW, K101 KEYSW, K102 KEYSW, K103 KEYSW, K104 KEYSW, K105 KEYSW, K106 KEYSW, K107 KEYSW, K108 KEYSW, K109 KEYSW, K110 KEYSW, K111 KEYSW, K200 KEYSW, K201 KEYSW, K202 KEYSW, K203 KEYSW, K204 KEYSW, K205 KEYSW, K206 KEYSW, K207 KEYSW, K208 KEYSW, K209 KEYSW, K210 KEYSW, K211 KEYSW, K303 KEYSW, K304 KEYSW, K305 KEYSW, K306 KEYSW, K307 KEYSW, K308 KEYSW, U0 ProMicro

Commit message: Add Opus revA files
Parts:
- added MH0, MH1, MH2, MH3, MH4, MH5: MountingHole_Pad, MountingHole:MountingHole_2.2mm_M2_Pad, symbol Mechanical:MountingHole_Pad
- D000, D001, D002, D003, D004, D005, D006, D007, D008, D009, D010, D011, D100, D101, D102, D103, D104, D105, D106, D107, D108, D109, D110, D111, D200, D201, D202, D203, D204, D205, D206, D207, D208, D209, D210, D211, D303, D304, D305, D306, D307, D308: footprint Diode_THT:D_DO-35_SOD27_P7.62mm_Horizontal -> Keebio-Parts:Diode-dual
- K000, K001, K002, K003, K004, K005, K006, K007, K008, K009, K010, K011, K100, K101, K102, K103, K104, K105, K106, K107, K108, K109, K110, K111, K200, K201, K202, K203, K204, K205, K206, K207, K208, K209, K210, K211, K303, K304, K305, K306, K307, K308: footprint (none) -> MX_Only:MXOnly-1U-Hotswap-Antishear
- U0: footprint (none) -> Keebio-Parts:Elite-C
Connections:
- no-connect marks 5 -> 11
