File: opus/pcb/opus.kicad_pcb (KiCad board)
At the start: 2 copper layers, 301.6 x 116.9 mm, 91 parts, among them K000 KEYSW, K001 KEYSW, K002 KEYSW, K003 KEYSW, K004 KEYSW, K005 KEYSW, K006 KEYSW, K007 KEYSW, K008 KEYSW, K009 KEYSW, K010 KEYSW, K011 KEYSW, K100 KEYSW, K101 KEYSW, K102 KEYSW, K103 KEYSW, K104 KEYSW, K105 KEYSW, K106 KEYSW, K107 KEYSW, K108 KEYSW, K109 KEYSW, K110 KEYSW, K111 KEYSW, K200 KEYSW, K201 KEYSW, K202 KEYSW, K203 KEYSW, K204 KEYSW, K205 KEYSW, K206 KEYSW, K207 KEYSW, K208 KEYSW, K209 KEYSW, K210 KEYSW, K211 KEYSW, K303 KEYSW, K304 KEYSW, K305 KEYSW, K306 KEYSW, K307 KEYSW, K308 KEYSW, U0 ProMicro

Commit message: Add Opus revB with col6 fix
Routing:
- net col6: track 140.2 -> 154.5 mm
Other:
- board text added: "Opus revB"
- board text removed: "Opus revA"
Changed lines of the file:
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@@
     (thickness 1.6)
     (drawings 664)
-    (tracks 632)
+    (tracks 634)
     (zones 0)
     (modules 91)
@@
     (visible_elements 7FFFFFFF)
     (pcbplotparams
-      (layerselection 0x010fc_ffffffff)
-      (usegerberextensions false)
+      (layerselection 0x010f0_ffffffff)
+      (usegerberextensions true)
       (usegerberattributes false)
       (usegerberadvancedattributes false)
@@
       (plotinvisibletext false)
       (padsonsilk false)
-      (subtractmaskfromsilk false)
+      (subtractmaskfromsilk true)
       (outputformat 1)
       (mirror false)
-      (drillshape 1)
+      (drillshape 0)
       (scaleselection 1)
       (outputdirectory ""))
@@
     (pad 2 smd rect (at 5.842 -5.08 353) (size 4.5 2.5) (layers B.Cu)
       (net 49 col2))
-    (pad 1 smd rect (at -7.085 -2.540002 353) (size 4.5 2.5) (layers B.Cu)
+    (pad 1 smd rect (at -7.085 -2.540003 353) (size 4.5 2.5) (layers B.Cu)
       (net 4 "Net-(D002-Pad2)"))
     (pad 2 thru_hole circle (at 7.62 -4.318 353) (size 0.8 0.8) (drill 0.4) (layers *.Cu)
@@
     (pad 2 smd rect (at 5.815 -5.08 353) (size 2.55 2.5) (layers B.Paste B.Mask)
       (net 49 col2))
-    (pad 1 smd rect (at -7.085 -2.540002 353) (size 2.55 2.5) (layers B.Paste B.Mask)
+    (pad 1 smd rect (at -7.085 -2.540003 353) (size 2.55 2.5) (layers B.Paste B.Mask)
       (net 4 "Net-(D002-Pad2)"))
     (pad "" np_thru_hole circle (at 5.08 0 41.0996) (size 1.75 1.75) (drill 1.75) (layers *.Cu *.Mask))
@@
     (pad 2 thru_hole circle (at 7.62 -5.842 350) (size 0.8 0.8) (drill 0.4) (layers *.Cu)
       (net 51 col4))
-    (pad 1 thru_hole circle (at -8.889998 -1.778 350) (size 0.8 0.8) (drill 0.4) (layers *.Cu)
+    (pad 1 thru_hole circle (at -8.889997 -1.778 350) (size 0.8 0.8) (drill 0.4) (layers *.Cu)
       (net 6 "Net-(D004-Pad2)"))
     (pad 2 thru_hole circle (at 7.62 -4.318 350) (size 0.8 0.8) (drill 0.4) (layers *.Cu)
@@
     (pad 2 thru_hole circle (at 7.62 -5.842 350) (size 0.8 0.8) (drill 0.4) (layers *.Cu)
       (net 52 col5))
-    (pad 1 thru_hole circle (at -8.889998 -1.778 350) (size 0.8 0.8) (drill 0.4) (layers *.Cu)
+    (pad 1 thru_hole circle (at -8.889997 -1.778 350) (size 0.8 0.8) (drill 0.4) (layers *.Cu)
       (net 7 "Net-(D005-Pad2)"))
     (pad 2 thru_hole circle (at 7.62 -4.318 350) (size 0.8 0.8) (drill 0.4) (layers *.Cu)
@@
       (net 10 "Net-(D008-Pad2)"))
     (pad "" np_thru_hole circle (at 0 0 8) (size 3.9878 3.9878) (drill 3.9878) (layers *.Cu *.Mask))
-    (pad 2 thru_hole circle (at 2.54 -5.079998 8) (size 4 4) (drill 3) (layers *.Cu)
+    (pad 2 thru_hole circle (at 2.54 -5.079997 8) (size 4 4) (drill 3) (layers *.Cu)
       (net 55 col8))
   )
@@
     (pad "" np_thru_hole circle (at -5.08 0 41.0996) (size 1.75 1.75) (drill 1.75) (layers *.Cu *.Mask))
     (pad "" np_thru_hole circle (at 5.08 0 41.0996) (size 1.75 1.75) (drill 1.75) (layers *.Cu *.Mask))
-    (pad 1 smd rect (at -7.085 -2.540002 353) (size 2.55 2.5) (layers B.Paste B.Mask)
+    (pad 1 smd rect (at -7.085 -2.540003 353) (size 2.55 2.5) (layers B.Paste B.Mask)
       (net 17 "Net-(D102-Pad2)"))
     (pad 2 smd rect (at 5.815 -5.08 353) (size 2.55 2.5) (layers B.Paste B.Mask)
@@
     (pad 2 thru_hole circle (at 7.62 -4.318 353) (size 0.8 0.8) (drill 0.4) (layers *.Cu)
       (net 49 col2))
-    (pad 1 smd rect (at -7.085 -2.540002 353) (size 4.5 2.5) (layers B.Cu)
+    (pad 1 smd rect (at -7.085 -2.540003 353) (size 4.5 2.5) (layers B.Cu)
       (net 17 "Net-(D102-Pad2)"))
     (pad 2 smd rect (at 5.842 -5.08 353) (size 4.5 2.5) (layers B.Cu)
@@
     (pad 2 thru_hole circle (at 7.62 -5.842 350) (size 0.8 0.8) (drill 0.4) (layers *.Cu)
       (net 51 col4))
-    (pad 1 thru_hole circle (at -8.889998 -1.778 350) (size 0.8 0.8) (drill 0.4) (layers *.Cu)
+    (pad 1 thru_hole circle (at -8.889997 -1.778 350) (size 0.8 0.8) (drill 0.4) (layers *.Cu)
       (net 19 "Net-(D104-Pad2)"))
     (pad 2 thru_hole circle (at 7.62 -4.318 350) (size 0.8 0.8) (drill 0.4) (layers *.Cu)
@@
     (pad 2 thru_hole circle (at 7.62 -4.318 350) (size 0.8 0.8) (drill 0.4) (layers *.Cu)
       (net 52 col5))
-    (pad 1 thru_hole circle (at -8.889998 -1.778 350) (size 0.8 0.8) (drill 0.4) (layers *.Cu)
+    (pad 1 thru_hole circle (at -8.889997 -1.778 350) (size 0.8 0.8) (drill 0.4) (layers *.Cu)
       (net 20 "Net-(D105-Pad2)"))
     (pad 2 thru_hole circle (at 7.62 -5.842 350) (size 0.8 0.8) (drill 0.4) (layers *.Cu)
@@
       (net 23 "Net-(D108-Pad2)"))
     (pad "" np_thru_hole circle (at 0 0 8) (size 3.9878 3.9878) (drill 3.9878) (layers *.Cu *.Mask))
-    (pad 2 thru_hole circle (at 2.54 -5.079998 8) (size 4 4) (drill 3) (layers *.Cu)
+    (pad 2 thru_hole circle (at 2.54 -5.079997 8) (size 4 4) (drill 3) (layers *.Cu)
       (net 55 col8))
   )
@@
     (pad 2 smd rect (at 5.842 -5.08 353) (size 4.5 2.5) (layers B.Cu)
       (net 49 col2))
-    (pad 1 smd rect (at -7.085 -2.540002 353) (size 4.5 2.5) (layers B.Cu)
+    (pad 1 smd rect (at -7.085 -2.540003 353) (size 4.5 2.5) (layers B.Cu)
       (net 30 "Net-(D202-Pad2)"))
     (pad 2 thru_hole circle (at 7.62 -4.318 353) (size 0.8 0.8) (drill 0.4) (layers *.Cu)
@@
     (pad 2 smd rect (at 5.815 -5.08 353) (size 2.55 2.5) (layers B.Paste B.Mask)
       (net 49 col2))
-    (pad 1 smd rect (at -7.085 -2.540002 353) (size 2.55 2.5) (layers B.Paste B.Mask)
+    (pad 1 smd rect (at -7.085 -2.540003 353) (size 2.55 2.5) (layers B.Paste B.Mask)
       (net 30 "Net-(D202-Pad2)"))
     (pad "" np_thru_hole circle (at 5.08 0 41.0996) (size 1.75 1.75) (drill 1.75) (layers *.Cu *.Mask))
@@
     (pad 2 thru_hole circle (at 7.62 -4.318 350) (size 0.8 0.8) (drill 0.4) (layers *.Cu)
       (net 51 col4))
-    (pad 1 thru_hole circle (at -8.889998 -1.778 350) (size 0.8 0.8) (drill 0.4) (layers *.Cu)
+    (pad 1 thru_hole circle (at -8.889997 -1.778 350) (size 0.8 0.8) (drill 0.4) (layers *.Cu)
       (net 32 "Net-(D204-Pad2)"))
     (pad 2 thru_hole circle (at 7.62 -5.842 350) (size 0.8 0.8) (drill 0.4) (layers *.Cu)
@@
     (pad 2 thru_hole circle (at 7.62 -5.842 350) (size 0.8 0.8) (drill 0.4) (layers *.Cu)
       (net 52 col5))
-    (pad 1 thru_hole circle (at -8.889998 -1.778 350) (size 0.8 0.8) (drill 0.4) (layers *.Cu)
+    (pad 1 thru_hole circle (at -8.889997 -1.778 350) (size 0.8 0.8) (drill 0.4) (layers *.Cu)
       (net 33 "Net-(D205-Pad2)"))
     (pad 2 thru_hole circle (at 7.62 -4.318 350) (size 0.8 0.8) (drill 0.4) (layers *.Cu)
@@
     (fp_line (start 9.525 9.525) (end -9.525 9.525) (layer Dwgs.User) (width 0.15))
     (fp_line (start -9.525 9.525) (end -9.525 -9.525) (layer Dwgs.User) (width 0.15))
-    (pad 2 thru_hole circle (at 2.54 -5.079998 8) (size 4 4) (drill 3) (layers *.Cu)
+    (pad 2 thru_hole circle (at 2.54 -5.079997 8) (size 4 4) (drill 3) (layers *.Cu)
       (net 55 col8))
     (pad "" np_thru_hole circle (at 0 0 8) (size 3.9878 3.9878) (drill 3.9878) (layers *.Cu *.Mask))
@@
   (gr_line (start 307.499708 185.038449) (end 314.686042 177.852115) (layer F.SilkS) (width 0.2))
   (gr_line (start 310.7944 183.642) (end 308.799474 185.636925) (layer F.SilkS) (width 0.2))
-  (gr_text "Opus revA" (at 314.96 191.1096) (layer F.SilkS)
+  (gr_text "Opus revB" (at 314.96 191.1096) (layer F.SilkS)
     (effects (font (size 1.5 1.5) (thickness 0.3)))
   )
@@
   (segment (start 339.4554 202.813791) (end 345.900217 196.368974) (width 0.25) (layer B.Cu) (net 53))
   (segment (start 345.900217 196.368974) (end 354.963426 196.368974) (width 0.25) (layer B.Cu) (net 53))
-  (via (at 369.331522 181.575537) (size 0.8) (drill 0.4) (layers F.Cu B.Cu) (net 53))
-  (segment (start 369.331522 182.000878) (end 369.331522 181.575537) (width 0.25) (layer F.Cu) (net 53))
-  (segment (start 364.148201 187.184199) (end 369.331522 182.000878) (width 0.25) (layer F.Cu) (net 53))
   (segment (start 361.093999 187.184199) (end 364.148201 187.184199) (width 0.25) (layer F.Cu) (net 53))
   (segment (start 358.3813 192.9511) (end 358.3813 189.896898) (width 0.25) (layer F.Cu) (net 53))
   (segment (start 358.3813 189.896898) (end 361.093999 187.184199) (width 0.25) (layer F.Cu) (net 53))
+  (via (at 369.316 181.7624) (size 0.8) (drill 0.4) (layers F.Cu B.Cu) (net 53))
+  (segment (start 364.148201 187.184199) (end 369.316 182.0164) (width 0.25) (layer F.Cu) (net 53))
+  (segment (start 369.316 182.0164) (end 369.316 181.7624) (width 0.25) (layer F.Cu) (net 53))
+  (segment (start 369.316 170.18313) (end 367.298634 168.165764) (width 0.25) (layer B.Cu) (net 53))
+  (segment (start 369.316 181.7624) (end 369.316 170.18313) (width 0.25) (layer B.Cu) (net 53))
   (segment (start 309.143399 163.080699) (end 308.2671 162.2044) (width 0.25) (layer B.Cu) (net 54))
   (segment (start 336.745198 190.682498) (end 309.143399 163.080699) (width 0.25) (layer B.Cu) (net 54))
