File: fernet/pcb/fernet/fernet.sch (KiCad schematic (older format))
At the start: 163 parts, among them SW0 Rotary_Encoder_Switch, SW1 Rotary_Encoder_Switch, SW2 Rotary_Encoder_Switch, U0 Elite-C

Commit message: Add 2u backspace support to fernet
Parts:
- added K_BKSPC2: KEYSW, MX_Only:MXOnly-2U-NoLED, symbol MX_Alps_Hybrid:MX-NoLED
Connections:
- net col14: now also K_BKSPC2.1 (COL)
- net at D_DEL1.2 (A), K_DEL1.2 (ROW): now also K_BKSPC2.2 (ROW)
Changed lines of the file:
@@
 	16150 3550 16150 3950
 Wire Wire Line
-	16150 1650 16150 2950
+	16150 1650 16150 2850
 $Comp
 L MX_Alps_Hybrid:MX-NoLED K_DEL1
@@
 Wire Wire Line
 	17450 5050 17450 4800
+$Comp
+L MX_Alps_Hybrid:MX-NoLED K_BKSPC2
+U 1 1 5EDFF8B6
+P 15500 3000
+F 0 "K_BKSPC2" H 15500 3233 60  0000 C CNN
+F 1 "KEYSW" H 15500 2900 60  0001 C CNN
+F 2 "MX_Only:MXOnly-2U-NoLED" H 15500 3000 60  0001 C CNN
+F 3 "" H 15500 3000 60  0000 C CNN
+	1    15500 3000
+	1    0    0    -1
+$EndComp
+Wire Wire Line
+	15850 2950 15850 2850
+Wire Wire Line
+	15850 2850 16150 2850
+Wire Wire Line
+	15650 2950 15850 2950
+Connection ~ 16150 2850
+Wire Wire Line
+	16150 2850 16150 2950
+Wire Wire Line
+	15450 3150 15700 3150
+Connection ~ 15700 3150
 $EndSCHEMATC
