File: fernet/pcb/fernet/fernet.kicad_pcb (KiCad board)
At the start: 2 copper layers, 320.5 x 127.5 mm, 165 parts, among them SW0 Rotary_Encoder_Switch, SW1 Rotary_Encoder_Switch, SW2 Rotary_Encoder_Switch, U0 Elite-C

Commit message: Fix missing fernet logo
Parts:
- added G***: LOGO, fernet:fernet_icon, F.Cu at (322.9, 37.5)
Changed lines of the file:
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@@
     (tracks 770)
     (zones 0)
-    (modules 165)
+    (modules 166)
     (nets 107)
   )
   (page A2)
   (layers
-    (0 F.Cu signal)
+    (0 F.Cu signal hide)
     (31 B.Cu signal)
     (32 B.Adhes user)
@@
     (add_net row5)
   )
+  (module fernet:fernet_icon (layer F.Cu)
+    (at 322.95 37.5)
+    (fp_text reference G*** (at 0 0) (layer F.SilkS) hide
+      (effects (font (size 1.524 1.524) (thickness 0.3)))
+    )
+    (fp_text value LOGO (at 0.75 0) (layer F.SilkS) hide
+      (effects (font (size 1.524 1.524) (thickness 0.3)))
+    )
+    (fp_poly (pts (xy 12.566316 -13.175536) (xy 11.164994 -13.009571) (xy 9.380998 -12.571453) (xy 7.590745 -11.729072)
+      (xy 5.975175 -10.579066) (xy 5.204876 -9.82636) (xy 3.958056 -8.439595) (xy 4.719554 -8.192201)
+      (xy 5.499119 -7.851711) (xy 6.238566 -7.414143) (xy 6.99608 -6.883479) (xy 5.843524 -5.709109)
+      (xy 5.030523 -4.980455) (xy 4.456641 -4.688952) (xy 4.283905 -4.704019) (xy 3.498191 -4.968565)
+      (xy 2.962066 -4.952209) (xy 2.585295 -4.746423) (xy 2.315494 -4.506356) (xy 2.26097 -4.229358)
+      (xy 2.437737 -3.761029) (xy 2.750181 -3.156618) (xy 3.198438 -2.256688) (xy 3.578031 -1.398916)
+      (xy 3.693609 -1.096682) (xy 3.98271 -0.267368) (xy 9.357895 -0.267368) (xy 9.357895 1.470527)
+      (xy 9.348655 2.404014) (xy 9.285577 2.923856) (xy 9.11562 3.151146) (xy 8.785745 3.206974)
+      (xy 8.596673 3.208421) (xy 7.835451 3.208421) (xy 8.526313 4.604399) (xy 9.048105 6.16603)
+      (xy 9.240693 7.941868) (xy 9.100505 9.721966) (xy 8.639563 11.262201) (xy 7.548031 13.060784)
+      (xy 6.092172 14.497174) (xy 4.337584 15.526621) (xy 2.349865 16.104378) (xy 1.393334 16.205257)
+      (xy 0.360246 16.21985) (xy -0.545408 16.168019) (xy -1.069474 16.075459) (xy -2.82786 15.268238)
+      (xy -4.418134 14.105121) (xy -5.729173 12.690702) (xy -6.649855 11.129578) (xy -6.832417 10.651015)
+      (xy -7.197185 8.739802) (xy -7.181649 8.465818) (xy -3.729116 8.465818) (xy -3.653052 9.079477)
+      (xy -3.62838 9.21746) (xy -3.238075 10.204125) (xy -2.513482 11.21479) (xy -1.610938 12.060776)
+      (xy -0.94076 12.461088) (xy 0.224987 12.758174) (xy 1.578947 12.793371) (xy 2.839907 12.560891)
+      (xy 2.901155 12.540161) (xy 3.473628 12.266406) (xy 3.740612 11.992564) (xy 3.743158 11.970152)
+      (xy 3.534526 11.565644) (xy 2.987969 10.98549) (xy 2.222499 10.33181) (xy 1.357126 9.706726)
+      (xy 0.555038 9.234498) (xy -0.197033 8.917233) (xy -1.130941 8.610177) (xy -2.09837 8.350505)
+      (xy -2.951003 8.17539) (xy -3.540524 8.122007) (xy -3.70841 8.165916) (xy -3.729116 8.465818)
+      (xy -7.181649 8.465818) (xy -7.08587 6.776794) (xy -6.529702 4.879244) (xy -6.377084 4.609375)
+      (xy -2.524663 4.609375) (xy -0.512359 5.189782) (xy 1.881363 6.07946) (xy 3.944127 7.294263)
+      (xy 4.812632 7.975709) (xy 5.748421 8.771068) (xy 5.833735 7.974477) (xy 5.760479 7.229927)
+      (xy 5.465749 6.299) (xy 5.298998 5.928803) (xy 4.386605 4.628406) (xy 3.196125 3.743128)
+      (xy 1.813616 3.2965) (xy 0.325136 3.312053) (xy -1.183257 3.813319) (xy -1.596542 4.04336)
+      (xy -2.524663 4.609375) (xy -6.377084 4.609375) (xy -5.559912 3.164402) (xy -4.535822 2.028541)
+      (xy -3.462267 1.196677) (xy -2.310878 0.528662) (xy -1.24391 0.108251) (xy -0.617358 0.005872)
+      (xy -0.017199 -0.133722) (xy 0.149915 -0.559984) (xy -0.043786 -1.192484) (xy -0.361733 -1.890303)
+      (xy -1.517709 -0.755799) (xy -2.673684 0.378705) (xy -3.877839 -0.803083) (xy -5.081993 -1.984871)
+      (xy -3.864333 -3.221121) (xy -3.209473 -3.914053) (xy -2.927164 -4.383336) (xy -3.045426 -4.748184)
+      (xy -3.592279 -5.127809) (xy -4.411579 -5.549439) (xy -5.537535 -6.0145) (xy -6.829973 -6.345382)
+      (xy -8.386743 -6.556866) (xy -10.305695 -6.663734) (xy -11.923813 -6.68421) (xy -15.532885 -6.68421)
+      (xy -15.453284 -8.355263) (xy -15.373684 -10.026316) (xy -10.962105 -10.001496) (xy -8.754404 -9.95419)
+      (xy -6.96715 -9.823003) (xy -5.489268 -9.5826) (xy -4.20968 -9.207646) (xy -3.017313 -8.672804)
+      (xy -1.801089 -7.952739) (xy -1.704959 -7.89) (xy -0.335182 -6.991142) (xy 0.76576 -9.212935)
+      (xy 2.17366 -11.479732) (xy 3.954087 -13.368142) (xy 6.083793 -14.859366) (xy 8.539528 -15.934607)
+      (xy 9.39291 -16.18842) (xy 10.3827 -16.409684) (xy 11.310879 -16.549191) (xy 11.697369 -16.573669)
+      (xy 12.566316 -16.576842) (xy 12.566316 -13.175536)) (layer F.SilkS) (width 0.01))
+  )
   (module crossed_keys:crossed_keys_small (layer F.Cu)
